File: hardware/BREAD_Slice.kicad_pcb (KiCad board)
At the start: 2 copper layers, 70 x 100 mm, 15 parts, among them J1 Conn_01x10_Female

Commit message: removed old silk
Other:
- board text added: "BREAD Slice Template SLC_TEMP R3 04-2025"
- board text removed: "5V I2C Connector"
- board text removed: "BREAD Slice Template SLC_TEMP R0 20YY"
Changed lines of the file:
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@@
 		(tags "Arduino Nano")
 		(property "Reference" "A1"
-			(at -3.224 -2.364 0)
+			(at -0.035 -2.465 0)
 			(layer "F.SilkS")
 			(effects
@@
 		(attr smd)
 		(fp_text user "Heat Sink"
-			(at 0 -6.7 0)
+			(at -1.5 6.775 0)
 			(unlocked yes)
 			(layer "F.SilkS")
@@
 		)
 	)
-	(gr_text "5V I2C \nConnector"
-		(at 150.22 129.24 0)
-		(layer "B.SilkS")
-		(effects
-			(font
-				(size 1 1)
-				(thickness 0.15)
-			)
-			(justify bottom mirror)
-		)
-	)
 	(gr_text "GND"
 		(at 129.89619 88.522 0)
@@
 		)
 	)
-	(gr_text "BREAD Slice\nTemplate\nSLC_TEMP\nR0 20YY"
+	(gr_text "BREAD Slice\nTemplate\nSLC_TEMP\nR3 04-2025"
 		(at 128 103.5 270)
 		(layer "F.SilkS")
