File: hardware/BREAD_Slice.kicad_pcb (KiCad board)
At the start: 4 copper layers, 70 x 100 mm, 16 parts, among them J1 Conn_01x10_Female, U1 AP63205, U2 NUCLEO-L432KC

Commit message: review and revise board and update footprints
Parts:
- D1: footprint SparkFun-LED:WS2812-5050-4PIN -> KMLib_IC_SMD:WS2812-5050-4PIN
- HS1: footprint kml-custom:Thermal Pad -> KMLib_Mounting:Thermal Pad
- U2: footprint kml-custom:MODULE_NUCLEO-L432KC -> KMLib_Boards_Modules:MODULE_NUCLEO-L432KC
Routing:
- net /I2C_DAT: track 46.0 -> 49.9 mm
- net /I2C_CLK: track 46.3 -> 49.3 mm
- net +12V: track 48.2 -> 51.2 mm, vias 0 -> 1
