File: hardware/BREAD_Slice_Conn.kicad_sch (KiCad schematic)
At the start: 14 parts, among them J1 Conn_01x10_Female

Commit message: removed old silk
Parts:
- added J2, J3: Conn_01x08, TerminalBlock_4Ucon:TerminalBlock_4Ucon_1x08_P3.50mm_Horizontal, symbol Connector_Generic:Conn_01x08
Connections:
- net A0: now also J3.2 (Pin_2)
- net A1: now also J3.3 (Pin_3)
- net A2: now also J3.4 (Pin_4)
- net A3: now also J3.5 (Pin_5)
- net A6: now also J3.6 (Pin_6)
- net A7: now also J3.7 (Pin_7)
- net AREF: now also J3.1 (Pin_1)
- net D10: now also J2.4 (Pin_4)
- net D11: now also J2.3 (Pin_3)
- net D12: now also J2.2 (Pin_2)
- net D13: now also J2.1 (Pin_1)
- net D6: now also J2.8 (Pin_8)
- net D7: now also J2.7 (Pin_7)
- net D8: now also J2.6 (Pin_6)
- net D9: now also J2.5 (Pin_5)
- net RESET: now also J3.8 (Pin_8)
