File: hardware/BREAD_Slice_thProto.kicad_pcb (KiCad board)
At the start: 2 copper layers, 334 x 104.4 mm, 132 parts, among them J1 Conn_01x10_Female

Commit message: removed old silk
Parts:
- removed >NAME: >VALUE, kicad_wrk:USB_Mini-B-NOSILK
- removed the ? at (370.2, 123.8)
- removed the ? at (393.1, 121.3)
- removed the ? at (451.5, 98.4)
- removed the ? at (342.3, 65.4)
- removed the ? at (418.5, 111.1)
- removed the ? at (342.3, 95.9)
- removed the ? at (355.0, 68.0)
- removed the ? at (451.5, 47.6)
- removed the ? at (418.5, 103.5)
- removed the ? at (349.9, 123.8)
- removed the ? at (393.1, 141.6)
- removed the ? at (362.6, 123.8)
- removed the ? at (400.7, 52.7)
- removed the ? at (360.1, 54.0)
- removed the ? at (423.6, 88.3)
- removed the ? at (436.9, 131.5)
- removed the ? at (377.9, 123.8)
- removed the ? at (436.9, 141.6)
- removed the ? at (334.7, 123.8)
- removed the ? at (390.6, 123.8)
- removed the ? at (443.9, 73.7)
- removed the ? at (418.5, 123.8)
- removed the ? at (413.4, 98.4)
- removed the ? at (418.5, 128.9)
- removed the ? at (418.5, 136.5)
- removed the ? at (372.8, 123.8)
- removed the ? at (355.0, 54.0)
- removed the ? at (418.5, 113.7)
- removed the ? at (382.9, 123.8)
- removed the ? at (352.5, 123.8)
- removed the ? at (433.7, 55.3)
- removed the ? at (393.1, 111.1)
- removed the ? at (388.0, 78.1)
- removed the ? at (418.5, 126.4)
- removed the ? at (342.3, 70.5)
- removed the ? at (417.2, 51.5)
- removed the ? at (339.8, 123.8)
- removed the ? at (342.3, 75.6)
- removed the ? at (360.1, 46.4)
- removed the ? at (388.0, 123.8)
- removed the ? at (423.6, 98.4)
- removed the ? at (447.1, 131.5)
- removed the ? at (418.5, 139.1)
- removed the ? at (418.5, 134.0)
- removed the ? at (436.9, 121.3)
- removed the ? at (438.8, 85.7)
- removed the ? at (418.5, 106.1)
- removed the ? at (418.5, 108.6)
- removed the ? at (357.5, 123.8)
- removed the ? at (367.7, 123.8)
- removed the ? at (355.0, 98.4)
- removed the ? at (390.6, 52.7)
- removed the ? at (418.5, 121.3)
- removed the ? at (413.4, 88.3)
- removed the ? at (342.3, 80.7)
- removed the ? at (342.3, 68.0)
- removed the ? at (352.5, 54.0)
- removed the ? at (418.5, 118.8)
- removed the ? at (355.0, 123.8)
- removed the ? at (447.1, 141.6)
- removed the ? at (355.0, 88.3)
- removed the ? at (341.3, 47.5)
- removed the ? at (362.6, 54.0)
- removed the ? at (413.4, 78.1)
- removed the ? at (347.4, 123.8)
- removed the ? at (438.8, 95.9)
- removed the ? at (342.3, 73.0)
- removed the ? at (342.3, 88.3)
- removed the ? at (380.4, 123.8)
- removed the ? at (375.3, 123.8)
- removed the ? at (360.1, 123.8)
- removed the ? at (436.9, 73.7)
- removed the ? at (344.8, 123.8)
- removed the ? at (423.6, 78.1)
- removed the ? at (418.5, 141.6)
- removed the ? at (370.2, 52.7)
- removed the ? at (365.2, 123.8)
- removed the ? at (450.9, 73.7)
- removed the ? at (418.5, 131.5)
- removed the ? at (413.4, 68.0)
- removed the ? at (337.2, 123.8)
- removed the ? at (357.5, 54.0)
- removed the ? at (423.6, 68.0)
- removed the ? at (446.4, 62.9)
- removed the ? at (355.0, 78.1)
- removed the ? at (380.4, 52.7)
- removed the ? at (342.3, 123.8)
- removed the ? at (436.9, 111.1)
- removed the ? at (421.0, 57.8)
- removed the ? at (447.1, 121.3)
- removed the ? at (447.1, 111.1)
- removed the ? at (385.5, 123.8)
- removed the ? at (393.1, 131.5)
- removed the ? at (418.5, 116.2)
- removed G***: LOGO, kicad_wrk:LOGO_OPHW_600
- removed OLIMEX_LOGO**: OLIMEX_LOGO_TB, OLIMEX_LOGOs-FP:OLIMEX_LOGO_TB
- removed the REF** at (342.0, 62.9)
- removed the REF** at (345.9, 125.6)
- removed the REF** at (388.0, 78.1)
- removed RoHS: Compliant, OLIMEX_LOGOs-FP:LOGO_ROHS_1
Routing:
- net (no net): track 5927.6 -> 70.0 mm, vias 46 -> 0
- net GND: track 258.8 -> 364.3 mm
Other:
- board size 334 x 104.4 mm -> 70 x 100 mm
- board text added: "10"
- board text added: "11"
- board text added: "12"
- board text added: "13"
- board text added: "14"
- board text added: "15"
- board text added: "16"
- board text added: "17"
- board text added: "18"
- board text added: "19"
- board text added: "2"
- board text added: "20"
- board text added: "3"
- board text added: "4"
- board text added: "5"
- board text added: "6"
- board text added: "7"
- board text added: "8"
- board text added: "9"
- board text added: "BREAD Slice Template: -> thProto SLC_TEMP R2 04-2025"
- board text removed: "5V I2C Connector"
- board text removed: "BREAD Slice Template SLC_TEMP R0 20YY"
- board text removed: "SMT breadboard - Rev.A"
- board text removed: "http://www.olimex.com/"
