File: hardware-2layer/BREAD_Slice.kicad_pcb (KiCad board)
At the start: 2 copper layers, 70 x 100 mm, 22 parts, among them J1 Conn_01x10_Socket, SW1 SW_DIP_x04, U1 AP63205

Commit message: updated to add new one and keep current
Parts:
- removed ?: , 
- removed C5: 47u 25V, Capacitor_SMD:CP_Elec_6.3x7.7
- removed C6: 0.1u, Capacitor_SMD:C_0805_2012Metric_Pad1.18x1.45mm_HandSolder
- removed D2: WS2812B_5050, kml-custom:WS2812-5050-4PIN
- removed G***: LOGO, kml-custom:FAST-Logo-Medium
- removed Ref**: Val**, kml-custom:OSHW_Logo_8mm
- removed SW1: SW_DIP_x04, Button_Switch_SMD:SW_DIP_SPSTx04_Slide_9.78x12.34mm_W8.61mm_P2.54mm
- added Logo1: Logo_Open_Hardware_Small, Symbol:OSHW-Symbol_6.7x6mm_SilkScreen, F.Cu at (128.2, 71.9)
- A1: footprint kml-custom:Arduino_Nano_Headers -> Module:Arduino_Nano
- C1: value 10u -> 22uF
- D1: value 1N4007 -> WS2812B_5050; footprint Diode_SMD:D_SOD-123F -> SparkFun-LED:WS2812-5050-4PIN
- J1: value Conn_01x10_Socket -> Conn_01x10_Female
- U1: footprint kml-custom:SOIC_05WU-7_DIO-M -> Package_TO_SOT_SMD:TSOT-23-6
- moved D1 68.8 mm to (173.1, 135.7), turned to 0 degrees
Connections:
- net /slice_template/ESTOP renamed /ESTOP
- A1 pad 10: /slice_template/D7 -> unconnected-(A1-D7-Pad10)
- A1 pad 11: /slice_template/D8 -> unconnected-(A1-D8-Pad11)
- A1 pad 12: /slice_template/D9 -> unconnected-(A1-D9-Pad12)
- A1 pad 13: /slice_template/D10 -> unconnected-(A1-D10-Pad13)
- A1 pad 14: /slice_template/D11/MOSI -> unconnected-(A1-D11-Pad14)
- A1 pad 15: /slice_template/D12/MISO -> unconnected-(A1-D12-Pad15)
- A1 pad 16: /slice_template/D13/SCK -> unconnected-(A1-D13-Pad16)
- A1 pad 17: /slice_template/3V3 -> unconnected-(A1-3V3-Pad17)
- A1 pad 18: /slice_template/AREF -> unconnected-(A1-AREF-Pad18)
- A1 pad 19: /slice_template/A0 -> unconnected-(A1-A0-Pad19)
- A1 pad 20: /slice_template/A1 -> unconnected-(A1-A1-Pad20)
- A1 pad 21: /slice_template/A2 -> unconnected-(A1-A2-Pad21)
- A1 pad 22: /slice_template/A3 -> unconnected-(A1-A3-Pad22)
- A1 pad 23: /slice_template/I2C_DAT/A4 -> /I2C_DAT
- A1 pad 24: /slice_template/I2C_CLK/A5 -> /I2C_CLK
- A1 pad 25: /slice_template/A6 -> unconnected-(A1-A6-Pad25)
- A1 pad 26: /slice_template/A7 -> unconnected-(A1-A7-Pad26)
- A1 pad 28: /slice_template/~{RESET} -> unconnected-(A1-~{RESET}-Pad28)
- A1 pad 30: /slice_template/VIN -> unconnected-(A1-VIN-Pad30)
- A1 pad 6: /slice_template/SYNC/CAN_{INT} -> /INT
- A1 pad 7: /slice_template/INT/CAN_{CS} -> /SYNC
- A1 pad 8: /slice_template/LED -> /LED
- A1 pad 9: /slice_template/D6 -> unconnected-(A1-D6-Pad9)
- D1 pad 1: /slice_template/VIN -> +5V
- D1 pad 2: +12V -> unconnected-(D1-DOUT-Pad2)
- J1 pad 3: /slice_template/I2C_CLK -> /I2C_CLK
- J1 pad 4: /slice_template/I2C_DAT -> /I2C_DAT
- J1 pad 7: /slice_template/SYNC -> /INT
- J1 pad 8: /slice_template/INT -> /SYNC
Routing:
- net /slice_template/LED: track 92.9 -> 0.00 mm
- net /LED: track 0.00 -> 92.9 mm
- net /I2C_CLK: track 0.00 -> 46.3 mm
- net /I2C_DAT: track 0.00 -> 46.0 mm
- net GND: track 57.3 -> 16.8 mm, vias 19 -> 20
- net /slice_template/VIN: track 34.6 -> 0.00 mm
- net /slice_template/I2C_DAT/A4: track 31.1 -> 0.00 mm
- net /slice_template/I2C_CLK/A5: track 31.0 -> 0.00 mm
- net /SYNC: track 0.00 -> 23.7 mm
- net /INT: track 0.00 -> 23.3 mm
- net /slice_template/INT/CAN_{CS}: track 15.4 -> 0.00 mm
- net /slice_template/SYNC/CAN_{INT}: track 14.9 -> 0.00 mm
- net /slice_template/I2C_CLK: track 10.2 -> 0.00 mm
- net /slice_template/I2C_DAT: track 10.0 -> 0.00 mm
- net /slice_template/INT: track 6.49 -> 0.00 mm
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- added copper zone on B.Cu, net GNDPWR
